Commit message: fixing typo!

File: urdf/example.xacro (robot description, xacro)
@@ -3,5 +3,5 @@
   <!-- Import all sensors from sensors sub-folder -->
   <xacro:include filename="$(find logical_camera)/urdf/sensors/sensor_logical_camera.xacro" />
-  <xacro:kinect log_cam_name="log_cam_front"
+  <xacro:log_cam log_cam_name="log_cam_front"
           log_cam_px="0.5025"
           log_cam_py="0.0"

File: urdf/sensors/sensor_logical_camera.xacro (robot description, xacro)
@@ -7,5 +7,5 @@
   <xacro:macro name="log_cam"
     params="log_cam_name log_cam_px log_cam_py log_cam_pz log_cam_or log_cam_op log_cam_oy">
-    <link name="$(arg tf_prefix)${log_cam_name}_link">
+    <link name="$(arg tf_prefix)${log_cam_name}_link"/>
     <joint name="$(arg robot_name)_${log_cam_name}_joint" type="fixed">
       <parent link="$(arg tf_prefix)${log_cam_parent}" />
